Commit message: Add EE-space pipeline: kinematics, pipeline builders, and teleop/record/rollout examples

File: urdf/follower/TRLC-DK1-Follower.urdf (robot description, URDF)
Before this commit: robot TRLC-DK1-Follower, 11 links, 10 joints
Joints:
- removed joint joint1
- removed joint joint2
- removed joint joint3
- removed joint joint4
- removed joint joint5
- removed joint joint6
- added joint joint_1: type revolute, parent base_link, child link1-2, origin xyz=0 0 0.0615 rpy=0 0 0, axis 0 0 1, limit lower=-2.0943951023931953 upper=2.0943951023931953 effort=100 velocity=5.4
- added joint joint_2: type revolute, parent link1-2, child link2-3, origin xyz=0.02 0.0 0.0385 rpy=0 0 0, axis 0 1 0, limit lower=-0.08726646259971647 upper=3.141592653589793 effort=100 velocity=5.4
- added joint joint_3: type revolute, parent link2-3, child link3-4, origin xyz=-0.264 0 0 rpy=0 0 0, axis 0 -1 0, limit lower=-0.08726646259971647 upper=4.71238898038469 effort=100 velocity=5.4
- added joint joint_4: type revolute, parent link3-4, child link4-5, origin xyz=0.244004 0 0.059971 rpy=0 0 0, axis 0 -1 0, limit lower=-1.95 upper=1.5707963267948966 effort=20 velocity=5.4
- added joint joint_5: type revolute, parent link4-5, child link5-6, origin xyz=0.061868 0 0.0425 rpy=0 0 0, axis 0 0 -1, limit lower=-1.5707963267948966 upper=1.5707963267948966 effort=20 velocity=5.4
- added joint joint_6: type revolute, parent link5-6, child link6-7, origin xyz=0.032 0 -0.0425 rpy=0 0 0, axis 1 0 0, limit lower=-2.0943951023931953 upper=2.0943951023931953 effort=20 velocity=5.4
